Commit message: Added sensors to robot

File: catkin_ws/src/my_robot/urdf/my_robot.xacro (robot description, xacro)
@@ -1,4 +1,77 @@
 <?xml version='1.0'?>
 <robot name="my_robot" xmlns:xacro="http://www.ros.org/wiki/xacro">
+    <gazebo reference="left_wheel">
+    <material>Gazebo/Green</material>
+    </gazebo>
+    <gazebo reference="right_wheel">
+    <material>Gazebo/Green</material>
+    </gazebo>
+    <gazebo reference="chassis">
+    <material>Gazebo/Blue</material>
+    </gazebo>
+    <gazebo reference="camera">
+    <material>Gazebo/Red</material>
+    </gazebo>
+    <link name="hokuyo">
+    <pose> 0 0 0 0 0 0</pose>
+     <inertial>
+      <mass value="1e-5"/>
+      <origin xyz="0 0 0" rpy=" 0 0 0"/>
+      <inertia
+          ixx="1e-6" ixy="0" ixz="0"
+          iyy="1e-6" iyz="0"
+          izz="1e-6"
+      />
+    </inertial>
+    <collision name='collision'>
+      <origin xyz="0 0 0" rpy=" 0 0 0"/>
+      <geometry>
+         <box size="0.1 0.1 0.1"/>
+      </geometry>
+    </collision>
+    <visual name='visual'>
+    <origin xyz="0 0 0" rpy=" 0 0 0"/>
+    <geometry>
+    <mesh filename="package://my_robot/meshes/hokuyo.dae"/>
+    </geometry>
+    </visual>
+    </link>
+    <joint type="fixed" name="hokuyo_joint">
+    <origin xyz="0.15 0 0.1" rpy="0 0 0" />
+    <child link="hokuyo"/>
+    <parent link="chassis"/>
+    <axis xyz="0 1 0" rpy="0 0 0"/>
+    </joint>
+   <link name="camera">
+   <pose> 0 0 0 0 0 0</pose>
+    <inertial>
+      <mass value="0.1"/>
+      <origin xyz="0 0 0" rpy=" 0 0 0"/>
+      <inertia
+          ixx="1e-6" ixy="0" ixz="0"
+          iyy="1e-6" iyz="0"
+          izz="1e-6"
+      />
+      <box_inertia m="0.1" x="0.05"/>
+    </inertial>
+    <collision name='collision'>
+      <origin xyz="0 0 0" rpy=" 0 0 0"/>
+      <geometry>
+         <box size="0.05 0.05 0.05"/>
+      </geometry>
+    </collision>
+    <visual name='visual'>
+      <origin xyz="0 0 0" rpy=" 0 0 0"/>
+      <geometry>
+        <box size="0.05 0.05 0.05"/>
+      </geometry>
+    </visual>
+   </link>
+   <joint type="fixed" name="camera_joint">
+    <origin xyz="0.2 0 0" rpy="0 0 0" />
+    <child link="camera"/>
+    <parent link="chassis"/>
+    <axis xyz="0 1 0" rpy="0 0 0"/>
+    </joint>
     <link name="left_wheel">
     <pose>0 0 0 0 0 0</pose>

Commit message: Added sensor plugins, and also housed the robot inside a custom world.

File: catkin_ws/src/my_robot/urdf/my_robot.xacro (robot description, xacro)
@@ -1,4 +1,59 @@
 <?xml version='1.0'?>
 <robot name="my_robot" xmlns:xacro="http://www.ros.org/wiki/xacro">
+<xacro:include filename="$(find my_robot)/urdf/my_robot.gazebo" />
+  <link name="robot_footprint"></link>
+  <joint name="robot_footprint_joint" type="fixed">
+    <origin xyz="0 0 0" rpy="0 0 0" />
+    <parent link="robot_footprint"/>
+    <child link="chassis" />
+  </joint>
+  <link name='chassis'>
+    <pose>0 0 0.1 0 0 0</pose>
+    <inertial>
+      <mass value="15.0"/>
+      <origin xyz="0.0 0 0" rpy=" 0 0 0"/>
+      <inertia
+          ixx="0.1" ixy="0" ixz="0"
+          iyy="0.1" iyz="0"
+          izz="0.1"
+      />
+    </inertial>
+    <collision name='collision'>
+      <origin xyz="0 0 0" rpy=" 0 0 0"/>
+      <geometry>
+        <box size=".4 .2 .1"/>
+      </geometry>
+    </collision>
+    <visual name='chassis_visual'>
+      <origin xyz="0 0 0" rpy=" 0 0 0"/>
+      <geometry>
+        <box size=".4 .2 .1"/>
+      </geometry>
+    </visual>
+    <collision name='back_caster_collision'>
+      <origin xyz="-0.15 0 -0.05" rpy=" 0 0 0"/>
+      <geometry>
+        <sphere radius="0.0499"/>
+      </geometry>
+    </collision>
+    <visual name='back_caster_visual'>
+      <origin xyz="-0.15 0 -0.05" rpy=" 0 0 0"/>
+      <geometry>
+        <sphere radius="0.05"/>
+      </geometry>
+    </visual>
+    <collision name='front_caster_collision'>
+      <origin xyz="0.15 0 -0.05" rpy=" 0 0 0"/>
+      <geometry>
+        <sphere radius="0.0499"/>
+      </geometry>
+    </collision>
+    <visual name='front_caster_visual'>
+      <origin xyz="0.15 0 -0.05" rpy=" 0 0 0"/>
+      <geometry>
+        <sphere radius="0.05"/>
+      </geometry>
+    </visual>
+  </link>
     <gazebo reference="left_wheel">
     <material>Gazebo/Green</material>
@@ -53,5 +108,5 @@
           izz="1e-6"
       />
-      <box_inertia m="0.1" x="0.05"/>
+      <box_inertia m="0.1" x="0.05" y="0.05" z="0.05"/>
     </inertial>
     <collision name='collision'>
@@ -138,57 +193,3 @@
     <dynamics damping="1.0" friction="1.0"/>
     </joint>
-  <link name="robot_footprint"></link>
-  <joint name="robot_footprint_joint" type="fixed">
-    <origin xyz="0 0 0" rpy="0 0 0" />
-    <parent link="robot_footprint"/>
-    <child link="chassis" />
-  </joint>
-  <link name='chassis'>
-    <pose>0 0 0.1 0 0 0</pose>
-    <inertial>
-      <mass value="15.0"/>
-      <origin xyz="0.0 0 0" rpy=" 0 0 0"/>
-      <inertia
-          ixx="0.1" ixy="0" ixz="0"
-          iyy="0.1" iyz="0"
-          izz="0.1"
-      />
-    </inertial>
-    <collision name='collision'>
-      <origin xyz="0 0 0" rpy=" 0 0 0"/>
-      <geometry>
-        <box size=".4 .2 .1"/>
-      </geometry>
-    </collision>
-    <visual name='chassis_visual'>
-      <origin xyz="0 0 0" rpy=" 0 0 0"/>
-      <geometry>
-        <box size=".4 .2 .1"/>
-      </geometry>
-    </visual>
-    <collision name='back_caster_collision'>
-      <origin xyz="-0.15 0 -0.05" rpy=" 0 0 0"/>
-      <geometry>
-        <sphere radius="0.0499"/>
-      </geometry>
-    </collision>
-    <visual name='back_caster_visual'>
-      <origin xyz="-0.15 0 -0.05" rpy=" 0 0 0"/>
-      <geometry>
-        <sphere radius="0.05"/>
-      </geometry>
-    </visual>
-    <collision name='front_caster_collision'>
-      <origin xyz="0.15 0 -0.05" rpy=" 0 0 0"/>
-      <geometry>
-        <sphere radius="0.0499"/>
-      </geometry>
-    </collision>
-    <visual name='front_caster_visual'>
-      <origin xyz="0.15 0 -0.05" rpy=" 0 0 0"/>
-      <geometry>
-        <sphere radius="0.05"/>
-      </geometry>
-    </visual>
-  </link>
 </robot>

Commit message: finished tweaking process_image and robot model.

File: catkin_ws/src/my_robot/urdf/my_robot.xacro (robot description, xacro)
@@ -11,10 +11,10 @@
     <pose>0 0 0.1 0 0 0</pose>
     <inertial>
-      <mass value="15.0"/>
+      <mass value="10"/>
       <origin xyz="0.0 0 0" rpy=" 0 0 0"/>
       <inertia
-          ixx="0.1" ixy="0" ixz="0"
-          iyy="0.1" iyz="0"
-          izz="0.1"
+          ixx="0.08" ixy="0" ixz="0"
+          iyy="0.08" iyz="0"
+          izz="0.15"
       />
     </inertial>
@@ -22,5 +22,5 @@
       <origin xyz="0 0 0" rpy=" 0 0 0"/>
       <geometry>
-        <box size=".4 .2 .1"/>
+        <box size=".15 .1 .04"/>
       </geometry>
     </collision>
@@ -28,43 +28,43 @@
       <origin xyz="0 0 0" rpy=" 0 0 0"/>
       <geometry>
-        <box size=".4 .2 .1"/>
+        <box size=".15 .1 .04"/>
       </geometry>
     </visual>
     <collision name='back_caster_collision'>
-      <origin xyz="-0.15 0 -0.05" rpy=" 0 0 0"/>
+      <origin xyz="-0.07 0 -0.020" rpy=" 0 0 0"/>
       <geometry>
-        <sphere radius="0.0499"/>
+        <sphere radius="0.01"/>
       </geometry>
     </collision>
     <visual name='back_caster_visual'>
-      <origin xyz="-0.15 0 -0.05" rpy=" 0 0 0"/>
+      <origin xyz="-0.07 0 -0.020" rpy=" 0 0 0"/>
       <geometry>
-        <sphere radius="0.05"/>
+        <sphere radius="0.01"/>
       </geometry>
     </visual>
     <collision name='front_caster_collision'>
-      <origin xyz="0.15 0 -0.05" rpy=" 0 0 0"/>
+      <origin xyz="0.07 0 -0.020" rpy=" 0 0 0"/>
       <geometry>
-        <sphere radius="0.0499"/>
+        <sphere radius="0.01"/>
       </geometry>
     </collision>
     <visual name='front_caster_visual'>
-      <origin xyz="0.15 0 -0.05" rpy=" 0 0 0"/>
+      <origin xyz="0.07 0 -0.020" rpy=" 0 0 0"/>
       <geometry>
-        <sphere radius="0.05"/>
+        <sphere radius="0.01"/>
       </geometry>
     </visual>
   </link>
     <gazebo reference="left_wheel">
+    <material>Gazebo/White</material>
+    </gazebo>
+    <gazebo reference="right_wheel">
+    <material>Gazebo/White</material>
+    </gazebo>
+    <gazebo reference="chassis">
     <material>Gazebo/Green</material>
     </gazebo>
-    <gazebo reference="right_wheel">
-    <material>Gazebo/Green</material>
-    </gazebo>
-    <gazebo reference="chassis">
-    <material>Gazebo/Blue</material>
-    </gazebo>
     <gazebo reference="camera">
-    <material>Gazebo/Red</material>
+    <material>Gazebo/Black</material>
     </gazebo>
     <link name="hokuyo">
@@ -93,5 +93,5 @@
     </link>
     <joint type="fixed" name="hokuyo_joint">
-    <origin xyz="0.15 0 0.1" rpy="0 0 0" />
+    <origin xyz="0 0 0.025" rpy="0 0 0" />
     <child link="hokuyo"/>
     <parent link="chassis"/>
@@ -101,5 +101,5 @@
    <pose> 0 0 0 0 0 0</pose>
     <inertial>
-      <mass value="0.1"/>
+      <mass value="1e-5"/>
       <origin xyz="0 0 0" rpy=" 0 0 0"/>
       <inertia
@@ -113,5 +113,5 @@
       <origin xyz="0 0 0" rpy=" 0 0 0"/>
       <geometry>
-         <box size="0.05 0.05 0.05"/>
+         <box size="0.025 0.025 0.025"/>
       </geometry>
     </collision>
@@ -119,10 +119,10 @@
       <origin xyz="0 0 0" rpy=" 0 0 0"/>
       <geometry>
-        <box size="0.05 0.05 0.05"/>
+        <box size="0.025 0.025 0.025"/>
       </geometry>
     </visual>
    </link>
    <joint type="fixed" name="camera_joint">
-    <origin xyz="0.2 0 0" rpy="0 0 0" />
+    <origin xyz="0.075 0 0.0325" rpy="0 0 0" />
     <child link="camera"/>
     <parent link="chassis"/>
@@ -132,10 +132,10 @@
     <pose>0 0 0 0 0 0</pose>
     <inertial>
-      <mass value="5"/>
+      <mass value="1.5"/>
       <origin xyz="0 0 0" rpy=" 0 1.5707 1.5707"/>
       <inertia
-          ixx="0.1" ixy="0" ixz="0"
-          iyy="0.1" iyz="0"
-          izz="0.1"
+          ixx="0.01" ixy="0" ixz="0"
+          iyy="0.01" iyz="0"
+          izz="0.01"
       />
     </inertial>
@@ -143,5 +143,5 @@
       <origin xyz="0 0 0" rpy=" 0 1.5707 1.5707"/>
       <geometry>
-         <cylinder length="0.05" radius="0.1"/>
+         <cylinder length="0.015" radius="0.03"/>
       </geometry>
     </collision>
@@ -149,5 +149,5 @@
       <origin xyz="0 0 0" rpy=" 0 1.5707 1.5707"/>
       <geometry>
-        <cylinder length="0.05" radius="0.1"/>
+        <cylinder length="0.015" radius="0.03"/>
       </geometry>
     </visual>
@@ -156,10 +156,10 @@
     <pose>0 0 0 0 0 0</pose>
     <inertial>
-      <mass value="5"/>
+      <mass value="1.5"/>
       <origin xyz="0 0 0" rpy=" 0 1.5707 1.5707"/>
       <inertia
-          ixx="0.1" ixy="0" ixz="0"
-          iyy="0.1" iyz="0"
-          izz="0.1"
+          ixx="0.01" ixy="0" ixz="0"
+          iyy="0.01" iyz="0"
+          izz="0.01"
       />
     </inertial>
@@ -167,5 +167,5 @@
       <origin xyz="0 0 0" rpy=" 0 1.5707 1.5707"/>
       <geometry>
-         <cylinder length="0.05" radius="0.1"/>
+         <cylinder length="0.015" radius="0.03"/>
       </geometry>
     </collision>
@@ -173,22 +173,22 @@
       <origin xyz="0 0 0" rpy=" 0 1.5707 1.5707"/>
       <geometry>
-         <cylinder length="0.05" radius="0.1"/>
+         <cylinder length="0.015" radius="0.03"/>
       </geometry>
     </visual>
     </link>
    <joint type="continuous" name="left_wheel_hinge">
-    <origin xyz="0 0.15 0" rpy="0 0 0" />
+    <origin xyz="0 0.06 0" rpy="0 0 0" />
     <child link="left_wheel"/>
     <parent link="chassis"/>
     <axis xyz="0 1 0" rpy="0 0 0"/>
-    <limit effort="10000" velocity="1000"/>
+    <limit effort="10000" velocity="2000"/>
     <dynamics damping="1.0" friction="1.0"/>
     </joint>
     <joint type="continuous" name="right_wheel_hinge">
-    <origin xyz="0 -0.15 0" rpy="0 0 0" />
+    <origin xyz="0 -0.06 0" rpy="0 0 0" />
     <child link="right_wheel"/>
     <parent link="chassis"/>
     <axis xyz="0 1 0" rpy="0 0 0"/>
-    <limit effort="10000" velocity="1000"/>
+    <limit effort="10000" velocity="2000"/>
     <dynamics damping="1.0" friction="1.0"/>
     </joint>

Commit message: fixed robot design

File: catkin_ws/src/my_robot/urdf/my_robot.xacro (robot description, xacro)
@@ -11,10 +11,10 @@
     <pose>0 0 0.1 0 0 0</pose>
     <inertial>
-      <mass value="10"/>
+      <mass value="15.0"/>
       <origin xyz="0.0 0 0" rpy=" 0 0 0"/>
       <inertia
-          ixx="0.08" ixy="0" ixz="0"
-          iyy="0.08" iyz="0"
-          izz="0.15"
+          ixx="0.1" ixy="0" ixz="0"
+          iyy="0.1" iyz="0"
+          izz="0.1"
       />
     </inertial>
@@ -22,5 +22,5 @@
       <origin xyz="0 0 0" rpy=" 0 0 0"/>
       <geometry>
-        <box size=".15 .1 .04"/>
+        <box size=".3 .2 .1"/>
       </geometry>
     </collision>
@@ -28,29 +28,29 @@
       <origin xyz="0 0 0" rpy=" 0 0 0"/>
       <geometry>
-        <box size=".15 .1 .04"/>
+        <box size=".4 .2 .1"/>
       </geometry>
     </visual>
     <collision name='back_caster_collision'>
-      <origin xyz="-0.07 0 -0.020" rpy=" 0 0 0"/>
+      <origin xyz="-0.15 0 -0.05" rpy=" 0 0 0"/>
       <geometry>
-        <sphere radius="0.01"/>
+        <sphere radius="0.0499"/>
       </geometry>
     </collision>
     <visual name='back_caster_visual'>
-      <origin xyz="-0.07 0 -0.020" rpy=" 0 0 0"/>
+      <origin xyz="-0.15 0 -0.05" rpy=" 0 0 0"/>
       <geometry>
-        <sphere radius="0.01"/>
+        <sphere radius="0.05"/>
       </geometry>
     </visual>
     <collision name='front_caster_collision'>
-      <origin xyz="0.07 0 -0.020" rpy=" 0 0 0"/>
+      <origin xyz="0.15 0 -0.05" rpy=" 0 0 0"/>
       <geometry>
-        <sphere radius="0.01"/>
+        <sphere radius="0.0499"/>
       </geometry>
     </collision>
     <visual name='front_caster_visual'>
-      <origin xyz="0.07 0 -0.020" rpy=" 0 0 0"/>
+      <origin xyz="0.15 0 -0.05" rpy=" 0 0 0"/>
       <geometry>
-        <sphere radius="0.01"/>
+        <sphere radius="0.05"/>
       </geometry>
     </visual>
@@ -93,5 +93,5 @@
     </link>
     <joint type="fixed" name="hokuyo_joint">
-    <origin xyz="0 0 0.025" rpy="0 0 0" />
+    <origin xyz="0 0 0.1" rpy="0 0 0" />
     <child link="hokuyo"/>
     <parent link="chassis"/>
@@ -106,12 +106,11 @@
           ixx="1e-6" ixy="0" ixz="0"
           iyy="1e-6" iyz="0"
-          izz="1e-6"
-      />
-      <box_inertia m="0.1" x="0.05" y="0.05" z="0.05"/>
+          izz="1e-6"/>
+      <box_inertia m="1e-5" x="0.05" y="0.05" z="0.05"/>
     </inertial>
     <collision name='collision'>
       <origin xyz="0 0 0" rpy=" 0 0 0"/>
       <geometry>
-         <box size="0.025 0.025 0.025"/>
+         <box size="0.05 0.05 0.05"/>
       </geometry>
     </collision>
@@ -119,10 +118,10 @@
       <origin xyz="0 0 0" rpy=" 0 0 0"/>
       <geometry>
-        <box size="0.025 0.025 0.025"/>
+        <box size="0.05 0.05 0.05"/>
       </geometry>
     </visual>
    </link>
    <joint type="fixed" name="camera_joint">
-    <origin xyz="0.075 0 0.0325" rpy="0 0 0" />
+    <origin xyz="0.2 0 0.075" rpy="0 0 0" />
     <child link="camera"/>
     <parent link="chassis"/>
@@ -132,10 +131,10 @@
     <pose>0 0 0 0 0 0</pose>
     <inertial>
-      <mass value="1.5"/>
+      <mass value="5"/>
       <origin xyz="0 0 0" rpy=" 0 1.5707 1.5707"/>
       <inertia
-          ixx="0.01" ixy="0" ixz="0"
-          iyy="0.01" iyz="0"
-          izz="0.01"
+          ixx="0.1" ixy="0" ixz="0"
+          iyy="0.1" iyz="0"
+          izz="0.1"
       />
     </inertial>
@@ -143,5 +142,5 @@
       <origin xyz="0 0 0" rpy=" 0 1.5707 1.5707"/>
       <geometry>
-         <cylinder length="0.015" radius="0.03"/>
+         <cylinder length="0.05" radius="0.1"/>
       </geometry>
     </collision>
@@ -149,5 +148,5 @@
       <origin xyz="0 0 0" rpy=" 0 1.5707 1.5707"/>
       <geometry>
-        <cylinder length="0.015" radius="0.03"/>
+        <cylinder length="0.05" radius="0.1"/>
       </geometry>
     </visual>
@@ -156,10 +155,10 @@
     <pose>0 0 0 0 0 0</pose>
     <inertial>
-      <mass value="1.5"/>
+      <mass value="5"/>
       <origin xyz="0 0 0" rpy=" 0 1.5707 1.5707"/>
       <inertia
-          ixx="0.01" ixy="0" ixz="0"
-          iyy="0.01" iyz="0"
-          izz="0.01"
+          ixx="0.1" ixy="0" ixz="0"
+          iyy="0.1" iyz="0"
+          izz="0.1"
       />
     </inertial>
@@ -167,5 +166,5 @@
       <origin xyz="0 0 0" rpy=" 0 1.5707 1.5707"/>
       <geometry>
-         <cylinder length="0.015" radius="0.03"/>
+         <cylinder length="0.05" radius="0.1"/>
       </geometry>
     </collision>
@@ -173,22 +172,22 @@
       <origin xyz="0 0 0" rpy=" 0 1.5707 1.5707"/>
       <geometry>
-         <cylinder length="0.015" radius="0.03"/>
+         <cylinder length="0.05" radius="0.1"/>
       </geometry>
     </visual>
     </link>
    <joint type="continuous" name="left_wheel_hinge">
-    <origin xyz="0 0.06 0" rpy="0 0 0" />
+    <origin xyz="0.06 0.15 0" rpy="0 0 0" />
     <child link="left_wheel"/>
     <parent link="chassis"/>
     <axis xyz="0 1 0" rpy="0 0 0"/>
-    <limit effort="10000" velocity="2000"/>
+    <limit effort="10000" velocity="1000"/>
     <dynamics damping="1.0" friction="1.0"/>
     </joint>
     <joint type="continuous" name="right_wheel_hinge">
-    <origin xyz="0 -0.06 0" rpy="0 0 0" />
+    <origin xyz="0.06 -0.15 0" rpy="0 0 0" />
     <child link="right_wheel"/>
     <parent link="chassis"/>
     <axis xyz="0 1 0" rpy="0 0 0"/>
-    <limit effort="10000" velocity="2000"/>
+    <limit effort="10000" velocity="1000"/>
     <dynamics damping="1.0" friction="1.0"/>
     </joint>
